File: digital lockin.brd (EAGLE design)
At the start: 76.2 x 94.9 mm, 24 parts, among them IC1 OPA2650E, IC2 LM358D, T2 NPN, U2 RASPBERRY_PICOSMD-TH, U5 TL431AIDBZR

Commit message: Add files via upload
Parts:
- moved C1 24.6 mm to (68.8, 17.3)
- moved R5 17.7 mm to (68.8, 10.4)
- moved R3 16.8 mm to (68.8, 25.9), turned to 90 degrees
- moved R7 15.8 mm to (64.8, 6.10)
- moved R9 14.1 mm to (48.0, 16.3)
- moved C8 14.1 mm to (62.0, 17.8), turned to 270 degrees
- moved PD1 12.2 mm to (45.0, 26.7), turned to 270 degrees
- moved C3 8.19 mm to (64.8, 13.2), turned to 90 degrees
- moved C10 6.28 mm to (53.8, 11.2)
- moved C2 5.59 mm to (59.2, 6.35)
- moved R6 2.09 mm to (58.2, 19.8)
- moved IC1 1.14 mm to (59.9, 12.4)
Connections:
- removed net V+: IC1.8
- removed net V-: IC1.4
- new net N$1: C1.2, IC1.2, PD1.K, R3.1, R6.1
- new net N$11: C3.1, IC1.6, R7.1
- new net N$13: C3.2, IC1.7, R6.2
- new net N$15: R9.1
- new net N$2: C10.2, IC1.3, R9.2
- new net N$4: C8.2, IC1.8
- new net N$5: IC1.1
- new net N$6: C1.1, R3.2, R5.1
- new net N$7: C2.1, IC1.5, R5.2
- new net N$8: C2.2, R7.2
- net GND: now also C10.1, C8.1, IC1.4, PD1.A
Routing:
- net 3V3: track 0.00 -> 167.9 mm, vias 0 -> 4
- net 5V: track 0.00 -> 164.9 mm, vias 0 -> 6
- net ADCREF: track 0.00 -> 145.3 mm, vias 0 -> 4
- net LEDCTRL: track 0.00 -> 114.0 mm, vias 0 -> 4
- net ADCMID: track 0.00 -> 56.6 mm, vias 0 -> 3
- net N$1: track 0.00 -> 54.6 mm, vias 0 -> 2
- net N$13: track 0.00 -> 22.2 mm, vias 0 -> 2
- net N$10: track 0.00 -> 19.5 mm, vias 0 -> 2
- net N$9: track 0.00 -> 17.0 mm
- net N$7: track 0.00 -> 12.9 mm
- net N$11: track 0.00 -> 11.2 mm, vias 0 -> 2
- net N$2: track 0.00 -> 11.1 mm
- net N$20: track 0.00 -> 7.35 mm
- net N$8: track 0.00 -> 5.69 mm
- net N$3: track 0.00 -> 5.64 mm
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- added copper zone on layer 1, net GND
- added copper zone on layer 16, net GND

Commit message: Add files via upload
Routing:
- net ADCMID: track 56.6 -> 88.1 mm, vias 3 -> 4
- net N$6: track 4.96 -> 16.3 mm
- net 3V3: track 167.9 -> 169.0 mm
Changed lines of the file:
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@@
 <via x="26.924" y="46.228" extent="1-16" drill="0.35"/>
 <wire x1="26.924" y1="46.228" x2="26.924" y2="40.132" width="0.3048" layer="16"/>
-<wire x1="26.924" y1="40.132" x2="58.42" y2="40.132" width="0" layer="19" extent="16-16"/>
+<via x="26.924" y="40.132" extent="1-16" drill="0.35"/>
+<wire x1="26.924" y1="40.132" x2="58.42" y2="40.132" width="0.1524" layer="1"/>
 </signal>
 <signal name="GND" class="1" airwireshidden="yes">
@@
 <contactref element="C8" pad="1"/>
 <polygon width="0.3048" layer="1" spacing="2.54" pour="hatch">
-<vertex x="72.136" y="93.98"/>
-<vertex x="74.168" y="93.98"/>
+<vertex x="0.508" y="94.488"/>
+<vertex x="74.168" y="94.488"/>
 <vertex x="74.168" y="1.524"/>
 <vertex x="0.508" y="1.524"/>
-<vertex x="0.508" y="94.488"/>
-<vertex x="4.064" y="94.488"/>
-<vertex x="4.064" y="93.98"/>
 </polygon>
 <polygon width="0.3048" layer="16" spacing="2.54" pour="hatch">
@@
 <wire x1="71.12" y1="33.02" x2="71.12" y2="83.312" width="0.3048" layer="16"/>
 <via x="71.12" y="83.312" extent="1-16" drill="0.35"/>
-<wire x1="52.926" y1="83.058" x2="70.866" y2="83.058" width="0.3048" layer="1"/>
-<wire x1="70.866" y1="83.058" x2="71.12" y2="83.312" width="0.3048" layer="1"/>
-<wire x1="52.926" y1="83.058" x2="51.816" y2="83.058" width="0" layer="19" extent="1-1"/>
+<wire x1="71.12" y1="83.312" x2="70.866" y2="83.058" width="0.3048" layer="1"/>
+<wire x1="70.866" y1="83.058" x2="52.926" y2="83.058" width="0.3048" layer="1"/>
+<wire x1="52.324" y1="83.058" x2="51.816" y2="83.058" width="0.3048" layer="1"/>
+<wire x1="52.926" y1="83.058" x2="52.324" y2="83.058" width="0.3048" layer="1"/>
 </signal>
 <signal name="ADCREF">
@@
 <contactref element="IC2" pad="2"/>
 <contactref element="R1" pad="2"/>
-<wire x1="12.258" y1="48.005" x2="12.132" y2="47.879" width="0.3048" layer="1"/>
 <wire x1="12.258" y1="49.275" x2="12.132" y2="49.149" width="0.3048" layer="1"/>
 <wire x1="12.258" y1="52.324" x2="12.258" y2="49.275" width="0.3048" layer="1"/>
-<wire x1="12.132" y1="47.879" x2="12.132" y2="49.149" width="0.3048" layer="1"/>
 <wire x1="12.258" y1="52.324" x2="12.7" y2="52.766" width="0.3048" layer="1"/>
 <wire x1="12.7" y1="52.766" x2="12.7" y2="54.864" width="0.3048" layer="1"/>
@@
 <wire x1="52.926" y1="80.518" x2="68.326" y2="80.518" width="0.3048" layer="1"/>
 <wire x1="68.326" y1="80.518" x2="68.58" y2="80.264" width="0.3048" layer="1"/>
+<wire x1="12.132" y1="49.149" x2="12.132" y2="47.879" width="0.3048" layer="1"/>
 </signal>
 <signal name="LEDCTRL">
@@
 <wire x1="44.958" y1="25.4" x2="68.392" y2="25.4" width="0.3048" layer="1"/>
 <wire x1="68.392" y1="25.4" x2="68.834" y2="24.958" width="0.3048" layer="1"/>
-<wire x1="68.834" y1="24.958" x2="68.834" y2="18.222" width="0.3048" layer="1"/>
 <wire x1="58.166" y1="20.762" x2="66.294" y2="20.762" width="0.3048" layer="1"/>
 <wire x1="66.294" y1="20.762" x2="68.834" y2="18.222" width="0.3048" layer="1"/>
@@
 <wire x1="56.388" y1="12.7" x2="56.46" y2="12.772" width="0.3048" layer="1"/>
 <wire x1="56.46" y1="12.772" x2="57.831" y2="12.772" width="0.3048" layer="1"/>
+<wire x1="68.834" y1="18.222" x2="68.834" y2="24.958" width="0.3048" layer="1"/>
 </signal>
 <signal name="N$2">
@@
 <contactref element="R5" pad="1"/>
 <wire x1="68.834" y1="16.322" x2="68.834" y2="11.364" width="0.3048" layer="1"/>
-<wire x1="68.834" y1="16.322" x2="68.834" y2="26.858" width="0" layer="19" extent="1-1"/>
+<wire x1="68.834" y1="16.322" x2="68.834" y2="16.42686875" width="0.3048" layer="1"/>
+<wire x1="68.834" y1="26.75313125" x2="68.834" y2="26.858" width="0.3048" layer="1"/>
+<wire x1="68.834" y1="16.42686875" x2="69.8634" y2="17.45626875" width="0.3048" layer="1"/>
+<wire x1="69.8634" y1="25.72373125" x2="68.834" y2="26.75313125" width="0.3048" layer="1"/>
+<wire x1="69.8634" y1="17.45626875" x2="69.8634" y2="25.72373125" width="0.3048" layer="1"/>
 </signal>
 <signal name="N$7">
@@
 <contactref element="R9" pad="1"/>
 </signal>
-<signal name="N$14">
-<via x="54.864" y="9.652" extent="1-16" drill="0.35"/>
-</signal>
-<signal name="N$16">
-<via x="61.976" y="17.78" extent="1-16" drill="0.35"/>
-</signal>
 </signals>
